File: JIS60.sch (KiCad schematic (older format))
At the start: 21 parts, among them SW1 SW_Push, U1 ATmega32U4-MU, U2 PRTR5V0U2X, Y1 16MHz

Commit message: Update submod
Connections:
- net COL1: now also U1.19 (PD1); no longer U1.41 (PF0)
- net COL10: now also U1.38 (PF5); no longer U1.29 (PB5)
- net COL11: now also U1.37 (PF6); no longer U1.28 (PB4)
- net COL12: now also U1.36 (PF7); no longer U1.27 (PD7)
- net COL13: now also U1.32 (PC7); no longer U1.26 (PD6)
- net COL2: now also U1.21 (PD3); no longer U1.40 (PF1)
- net COL3: now also U1.22 (PD5); no longer U1.39 (PF4)
- net COL4: now also U1.25 (PD4); no longer U1.38 (PF5)
- net COL5: now also U1.26 (PD6); no longer U1.37 (PF6)
- net COL6: now also U1.31 (PC6); no longer U1.36 (PF7)
- net COL7: now also U1.41 (PF0); no longer U1.32 (PC7)
- net COL8: now also U1.40 (PF1); no longer U1.31 (PC6)
- net COL9: now also U1.39 (PF4); no longer U1.30 (PB6)
- net ROW0: now also U1.30 (PB6); no longer U1.25 (PD4)
- net ROW1: now also U1.29 (PB5); no longer U1.22 (PD5)
- net ROW2: now also U1.28 (PB4); no longer U1.21 (PD3)
- net ROW3: now also U1.27 (PD7); no longer U1.10 (PB2)
- net ROW4: now also U1.1 (PE6); no longer U1.11 (PB3)
- net USB+: now reaches R1.1, U1.4 (D+)
- net USB-: now reaches R3.1, U1.3 (D-)
Changed lines of the file:
@@
 	3675 6975 3925 6975
 Connection ~ 3925 6975
-Text GLabel 3000 4100 2    60   Input ~ 0
-ROW3
-Text GLabel 3000 4200 2    60   Input ~ 0
+Text GLabel 3000 6100 2    60   Input ~ 0
 ROW4
-Text GLabel 3000 5800 2    60   Input ~ 0
-COL12
+Text GLabel 3000 4900 2    60   Input ~ 0
+COL13
 Text GLabel 3000 5700 2    60   Input ~ 0
-COL13
-Text GLabel 3000 6700 2    60   Input ~ 0
 COL5
-Text GLabel 3000 6500 2    60   Input ~ 0
+Text GLabel 3000 5600 2    60   Input ~ 0
 COL3
-Text GLabel 3000 6400 2    60   Input ~ 0
+Text GLabel 3000 5400 2    60   Input ~ 0
 COL2
-Text GLabel 3000 6300 2    60   Input ~ 0
+Text GLabel 3000 5200 2    60   Input ~ 0
 COL1
 Text GLabel 3000 5300 2    60   Input ~ 0
 COL0
-Text GLabel 3000 4800 2    60   Input ~ 0
+Text GLabel 3000 6400 2    60   Input ~ 0
 COL8
-Text GLabel 3000 4900 2    60   Input ~ 0
-COL7
-Text GLabel 3000 6800 2    60   Input ~ 0
-COL6
+Text GLabel 3000 5500 2    60   Input ~ 0
+COL4
+Text GLabel 3000 6500 2    60   Input ~ 0
+COL9
 Text GLabel 3000 6600 2    60   Input ~ 0
-COL4
-Text GLabel 3000 4500 2    60   Input ~ 0
-COL9
-Text GLabel 3000 4400 2    60   Input ~ 0
 COL10
-Text GLabel 3000 4300 2    60   Input ~ 0
+Text GLabel 3000 6700 2    60   Input ~ 0
 COL11
-Text GLabel 3000 5500 2    60   Input ~ 0
-ROW0
-Text GLabel 3000 5600 2    60   Input ~ 0
-ROW1
 Wire Wire Line
 	3925 6975 4300 6975
@@
 Wire Wire Line
 	1650 3525 1650 3575
-Text GLabel 3000 5400 2    60   Input ~ 0
-ROW2
 $Comp
 L Type-C:HRO-TYPE-C-31-M-12 USB1
@@
 	1    0    0    -1
 $EndComp
+Text GLabel 1700 4900 1    50   Input ~ 0
+USB+
+Text GLabel 1700 5000 3    50   Input ~ 0
+USB-
+Text GLabel 3000 6800 2    60   Input ~ 0
+COL12
+Text GLabel 3000 5800 2    60   Input ~ 0
+ROW3
+Text GLabel 3000 4400 2    60   Input ~ 0
+ROW1
+Text GLabel 3000 4300 2    60   Input ~ 0
+ROW2
+Text GLabel 3000 4500 2    60   Input ~ 0
+ROW0
+Text GLabel 3000 6300 2    60   Input ~ 0
+COL7
+Text GLabel 3000 4800 2    60   Input ~ 0
+COL6
 $EndSCHEMATC
