File: JIS60.kicad_pcb (KiCad board)
At the start: 2 copper layers, 285 x 95.1 mm, 150 parts, among them SW1 SW_Push, U1 ATmega32U4-MU, U2 PRTR5V0U2X, Y1 16MHz

Commit message: Update submod
Parts:
- moved R4 152.2 mm to (240.1, 253.5)
- moved C2 145.6 mm to (238.2, 253.5), turned to 270 degrees
- moved C4 138.3 mm to (238.2, 259.7)
- moved C1 138.1 mm to (229.3, 251.4)
- moved U1 136.5 mm to (232.7, 256.9), turned to 90 degrees
- moved C7 130.9 mm to (232.0, 262.7), turned to 180 degrees
- moved Y1 126.7 mm to (224.7, 257.1), turned to 270 degrees
- moved C3 126.1 mm to (226.8, 261.3), turned to 180 degrees
- moved SW1 124.8 mm to (253.2, 258.0), turned to 180 degrees
- moved C5 123.9 mm to (221.0, 256.1), turned to 180 degrees
- moved C6 120.8 mm to (221.0, 258.2)
- moved R5 118.0 mm to (237.4, 262.4), turned to 0 degrees
- moved R1 108.1 mm to (213.6, 256.4), turned to 90 degrees
- moved R3 107.0 mm to (211.7, 256.4), turned to 90 degrees
- moved F1 57.8 mm to (149.2, 192.1), turned to 270 degrees
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Connections:
- net Net-(R1-Pad1) renamed USB+
- net Net-(R3-Pad1) renamed USB-
- K_#1 pad 1: COL1 -> Net-(D7-Pad2)
- K_#1 pad 2: Net-(D7-Pad2) -> COL1
- K_ESC1 pad 1: COL0 -> Net-(D2-Pad2)
- K_ESC1 pad 2: Net-(D2-Pad2) -> COL0
- K_H1 pad 1: COL6 -> Net-(D35-Pad2)
- K_H1 pad 2: Net-(D35-Pad2) -> COL6
- U1 pad 1: Net-(U1-Pad1) -> ROW4
- U1 pad 10: ROW3 -> Net-(U1-Pad10)
- U1 pad 11: ROW4 -> Net-(U1-Pad11)
- U1 pad 19: Net-(U1-Pad19) -> COL1
- U1 pad 21: ROW2 -> COL2
- U1 pad 22: ROW1 -> COL3
- U1 pad 25: ROW0 -> COL4
- U1 pad 26: COL13 -> COL5
- U1 pad 27: COL12 -> ROW3
- U1 pad 28: COL11 -> ROW2
- U1 pad 29: COL10 -> ROW1
- U1 pad 30: COL9 -> ROW0
- U1 pad 31: COL8 -> COL6
- U1 pad 32: COL7 -> COL13
- U1 pad 36: COL6 -> COL12
- U1 pad 37: COL5 -> COL11
- U1 pad 38: COL4 -> COL10
- U1 pad 39: COL3 -> COL9
- U1 pad 40: COL2 -> COL8
- U1 pad 41: COL1 -> COL7
Routing:
- net ROW4: track 0.00 -> 322.6 mm, vias 0 -> 6
- net ROW2: track 0.00 -> 315.3 mm, vias 0 -> 4
- net ROW0: track 0.00 -> 309.3 mm, vias 0 -> 2
- net COL13: track 0.00 -> 293.5 mm, vias 0 -> 5
- net ROW1: track 0.00 -> 290.0 mm, vias 0 -> 4
- net COL12: track 0.00 -> 281.0 mm, vias 0 -> 7
- net GND: track 0.00 -> 255.1 mm, vias 0 -> 6
- net COL11: track 0.00 -> 219.6 mm, vias 0 -> 5
- net ROW3: track 0.00 -> 207.0 mm
- net +5V: track 0.00 -> 200.4 mm, vias 0 -> 8
- net COL10: track 0.00 -> 196.9 mm, vias 0 -> 5
- net COL0: track 0.00 -> 189.4 mm, vias 0 -> 7
- net COL1: track 0.00 -> 172.9 mm, vias 0 -> 6
- net COL2: track 0.00 -> 162.4 mm, vias 0 -> 6
- net COL9: track 0.00 -> 159.1 mm, vias 0 -> 5
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- added copper zone on B.Cu, net Earth
Other:
- net class Earth: trace_width 0.5 -> 0.508
- net class USB added: clearance 0.1778, trace_width 0.261112, via_dia 0.6, via_drill 0.4
- board text added: "JP60 R0.1 20210717 | ai03.com"

Commit message: Finalize data
Parts:
- added G***: LOGO, locallib:ai-ring-6mm-Combined, F.Cu at (252.4, 258.0)
- added G***: LOGO, locallib:ai-ring-6mm-Combined, B.Cu at (296.9, 258.0)
- added K_SPC2: MX-NoLED, MX_Only:MXOnly-1U-Hotswap, F.Cu at (277.0, 258.0)
- moved D42 12.7 mm to (288.1, 259.6)
- moved R5 0.36 mm to (237.4, 262.7)
Connections:
- REF** pad 1: (no net) -> Earth
Routing:
- net Earth: track 19.4 -> 61.1 mm
- net COL7: track 124.0 -> 143.0 mm
- net Net-(D42-Pad2): track 5.89 -> 19.6 mm
- net ROW4: track 322.6 -> 328.0 mm
Other:
- board text added: "1.25U"
- board text added: "1.5U"
- board text added: "1.75U"
- board text added: "2.25U"
- board text added: "6U-CENTERED"
- board text added: "6U-OFFCENTER"
- board text added: "ISO-ENTER"
- board text added: "JP60"
- board text added: "JP60 R1.0 20210717 | ai03.com"
- board text added: "RESET"
- board text removed: "JP60 R0.1 20210717 | ai03.com"
