File: matrix.sch (KiCad schematic (older format))
At the start: 128 parts

Commit message: Update submod
Connections:
- net COL0: now also K_ESC1.2 (ROW); no longer K_ESC1.1 (COL)
- net COL1: now also K_#1.2 (ROW); no longer K_#1.1 (COL)
- net COL6: now also K_H1.2 (ROW); no longer K_H1.1 (COL)
- net at D2.2 (A): now also K_ESC1.1 (COL); no longer K_ESC1.2 (ROW)
- net at D7.2 (A): now also K_#1.1 (COL); no longer K_#1.2 (ROW)
- net at D35.2 (A): now also K_H1.1 (COL); no longer K_H1.2 (ROW)
Other:
- moved on the sheet: K_#1, K_ESC1, K_H1
Changed lines of the file:
@@
 L MX_Alps_Hybrid:MX-NoLED K_ESC1
 U 1 1 5D45F55D
-P 3000 2125
-F 0 "K_ESC1" H 3033 2348 60  0000 C CNN
-F 1 "MX-NoLED" H 3033 2274 20  0000 C CNN
-F 2 "MX_Only:MXOnly-1U-Hotswap" H 2375 2100 60  0001 C CNN
-F 3 "" H 2375 2100 60  0001 C CNN
-	1    3000 2125
+P 2925 2050
+F 0 "K_ESC1" H 2958 2273 60  0000 C CNN
+F 1 "MX-NoLED" H 2958 2199 20  0000 C CNN
+F 2 "MX_Only:MXOnly-1U-Hotswap" H 2300 2025 60  0001 C CNN
+F 3 "" H 2300 2025 60  0001 C CNN
+	1    2925 2050
 	1    0    0    -1
 $EndComp
@@
 	0    -1   -1   0
 $EndComp
-Wire Wire Line
-	2875 2275 2950 2275
-$Comp
-L MX_Alps_Hybrid:MX-NoLED K_#1
-U 1 1 5D45F56A
-P 3475 2125
-F 0 "K_#1" H 3508 2348 60  0000 C CNN
-F 1 "MX-NoLED" H 3508 2274 20  0000 C CNN
-F 2 "MX_Only:MXOnly-1U-Hotswap" H 2850 2100 60  0001 C CNN
-F 3 "" H 2850 2100 60  0001 C CNN
-	1    3475 2125
-	1    0    0    -1
-$EndComp
 $Comp
 L Device:D_Small D7
@@
 	0    -1   -1   0
 $EndComp
-Wire Wire Line
-	3350 2275 3425 2275
 $Comp
 L MX_Alps_Hybrid:MX-NoLED K_#2
@@
 	5250 3525 5325 3525
 $Comp
-L MX_Alps_Hybrid:MX-NoLED K_H1
-U 1 1 5D47FF41
-P 5850 3375
-F 0 "K_H1" H 5883 3598 60  0000 C CNN
-F 1 "MX-NoLED" H 5883 3524 20  0000 C CNN
-F 2 "MX_Only:MXOnly-1U-Hotswap" H 5225 3350 60  0001 C CNN
-F 3 "" H 5225 3350 60  0001 C CNN
-	1    5850 3375
-	1    0    0    -1
-$EndComp
-$Comp
 L Device:D_Small D35
 U 1 1 5D47FF47
@@
 	0    -1   -1   0
 $EndComp
-Wire Wire Line
-	5725 3525 5800 3525
 $Comp
 L MX_Alps_Hybrid:MX-NoLED K_J1
@@
 Wire Wire Line
 	6475 3950 6475 4575
-Wire Wire Line
-	6000 3950 6000 3325
 Connection ~ 6000 2700
 Wire Wire Line
 	6000 2700 6000 2075
-Connection ~ 6000 3325
-Wire Wire Line
-	6000 3325 6000 2700
 Wire Wire Line
 	5525 2075 5525 2700
@@
 Wire Wire Line
 	4100 3950 4100 3325
-Wire Wire Line
-	3625 2075 3625 2700
 Connection ~ 3625 2700
 Wire Wire Line
@@
 	3150 4575 3150 3950
 Connection ~ 3150 2700
-Wire Wire Line
-	3150 2700 3150 2075
 Connection ~ 3150 3950
 Connection ~ 2875 2475
@@
 Wire Wire Line
 	4100 2075 4100 1450
-Wire Wire Line
-	3150 2075 3150 1450
 Connection ~ 3625 3325
 $Comp
@@
 	1    0    0    -1
 $EndComp
-Connection ~ 3150 2075
 Connection ~ 4100 2075
 Connection ~ 4575 2075
@@
 Connection ~ 8375 2075
 Connection ~ 8850 2075
-Wire Wire Line
-	3625 2075 3625 1450
-Connection ~ 3625 2075
 $Comp
 L MX_Alps_Hybrid:MX-NoLED K_SRSFT1
@@
 	7625 4975 8100 4975
 Connection ~ 7900 3950
+$Comp
+L MX_Alps_Hybrid:MX-NoLED K_#1
+U 1 1 5D45F56A
+P 3400 2050
+F 0 "K_#1" H 3433 2273 60  0000 C CNN
+F 1 "MX-NoLED" H 3433 2199 20  0000 C CNN
+F 2 "MX_Only:MXOnly-1U-Hotswap" H 2775 2025 60  0001 C CNN
+F 3 "" H 2775 2025 60  0001 C CNN
+	1    3400 2050
+	1    0    0    -1
+$EndComp
+Wire Wire Line
+	3350 2200 3625 2200
+Wire Wire Line
+	3150 1450 3150 2200
+Wire Wire Line
+	3625 1450 3625 2200
+Connection ~ 3625 2200
+Wire Wire Line
+	3625 2200 3625 2700
+Wire Wire Line
+	2875 2200 3150 2200
+Connection ~ 3150 2200
+Wire Wire Line
+	3150 2200 3150 2700
+Wire Wire Line
+	3075 2000 3075 2275
+Wire Wire Line
+	2875 2275 3075 2275
+Wire Wire Line
+	3550 2000 3550 2275
+Wire Wire Line
+	3350 2275 3550 2275
+$Comp
+L MX_Alps_Hybrid:MX-NoLED K_H1
+U 1 1 5D47FF41
+P 5775 3300
+F 0 "K_H1" H 5808 3523 60  0000 C CNN
+F 1 "MX-NoLED" H 5808 3449 20  0000 C CNN
+F 2 "MX_Only:MXOnly-1U-Hotswap" H 5150 3275 60  0001 C CNN
+F 3 "" H 5150 3275 60  0001 C CNN
+	1    5775 3300
+	1    0    0    -1
+$EndComp
+Wire Wire Line
+	5925 3250 5925 3525
+Wire Wire Line
+	5725 3525 5925 3525
+Wire Wire Line
+	6000 2700 6000 3450
+Wire Wire Line
+	5725 3450 6000 3450
+Connection ~ 6000 3450
+Wire Wire Line
+	6000 3450 6000 3950
 $EndSCHEMATC

Commit message: Finalize data
Parts:
- added K_SPC2: MX-NoLED, MX_Only:MXOnly-1U-Hotswap, symbol MX_Alps_Hybrid:MX-NoLED
Connections:
- net COL7: now also K_SPC2.2 (ROW)
- net at D42.2 (A), K_SPC1.2 (ROW): now also K_SPC2.1 (COL)
Changed lines of the file:
@@
 Wire Wire Line
 	6000 3450 6000 3950
+$Comp
+L MX_Alps_Hybrid:MX-NoLED K_SPC2
+U 1 1 60F7C6E2
+P 5950 4625
+F 0 "K_SPC2" H 5983 4848 60  0000 C CNN
+F 1 "MX-NoLED" H 5983 4774 20  0000 C CNN
+F 2 "MX_Only:MXOnly-1U-Hotswap" H 5325 4600 60  0001 C CNN
+F 3 "" H 5325 4600 60  0001 C CNN
+	1    5950 4625
+	1    0    0    -1
+$EndComp
+Wire Wire Line
+	6200 4775 6100 4775
+Wire Wire Line
+	6100 4775 6100 4575
+Connection ~ 6200 4775
+Wire Wire Line
+	6475 4575 6475 4725
+Wire Wire Line
+	6475 4725 5900 4725
+Wire Wire Line
+	5900 4725 5900 4775
+Connection ~ 6475 4575
 $EndSCHEMATC
